Commit message: Added ros2_control

File: ros2_ws/src/cognibot_description/urdf/cognibot.urdf (robot description, URDF)
Before this commit: robot my_robot, 10 links, 9 joints
Links:
- removed link arm_base_link
- removed link camera_link
- removed link camera_link_optical
- removed link forearm_link
- removed link hand_link
Joints:
- removed joint arm_base_to_forearm_joint
- removed joint arm_base_to_mobile_base_joint
- removed joint base_camera_joint
- removed joint camera_optical_joint
- removed joint forearm_to_hand_joint
- joint base_caster_wheel_joint: origin xyz=-0.19999999999999998 0 -0.05 rpy=0 0 0 -> xyz=0.19999999999999998 0 -0.05 rpy=0 0 0

File: ros2_ws/src/cognibot_description/urdf/cognibot.urdf.xacro (robot description, xacro)
@@ -3,4 +3,6 @@
     <xacro:include filename="common_properties.xacro"/>
     <xacro:include filename="mobile_base.xacro"/>
+    <xacro:include filename="mobile_base_ros2_control.xacro"/>
+<!--
     <xacro:include filename="camera.xacro"/>
     <xacro:include filename="arm.xacro"/>
@@ -10,3 +12,4 @@
         <origin xyz="${base_length/3.0} 0 ${base_height}" rpy="0 0 0"/>
     </joint>
+     -->
 </robot>

File: ros2_ws/src/cognibot_description/urdf/mobile_base.xacro (robot description, xacro)
@@ -93,5 +93,5 @@
         <parent link="base_link"/>
         <child link="caster_wheel_link"/>
-        <origin xyz="${base_length/-3.0} 0 ${wheel_radius/-2.0}" rpy="0 0 0"/>
+        <origin xyz="${base_length/3.0} 0 ${wheel_radius/-2.0}" rpy="0 0 0"/>
     </joint>
 </robot>
