Commit message: Added LIDAR

File: ros2_ws/src/cognibot_description/urdf/camera.xacro (robot description, xacro)
@@ -24,9 +24,10 @@
         <origin xyz="${(base_length + camera_length) / 2.0} 0 ${base_height / 2.0}" rpy="0 0 0" />
     </joint>
-    <link name="camera_link_optical" />
+    <!-- <link name="camera_link_optical" /> -->
+<!--
     <joint name="camera_optical_joint" type="fixed">
         <origin xyz="0 0 0" rpy="${-pi/2} 0 ${-pi/2}"/>
         <parent link="camera_link"/>
         <child link="camera_link_optical"/>
-    </joint>
+    </joint> -->
 </robot>

File: ros2_ws/src/cognibot_description/urdf/cognibot.urdf.xacro (robot description, xacro)
@@ -3,5 +3,6 @@
     <xacro:include filename="common_properties.xacro"/>
     <xacro:include filename="mobile_base.xacro"/>
-    <xacro:include filename="mobile_base_ros2_control.xacro"/>
+    <!-- <xacro:include filename="mobile_base_ros2_control.xacro"/> -->
+    <xacro:include filename="camera.xacro"/>
 <!--
     <xacro:include filename="camera.xacro"/>
