Commit message: Implemented Basic TEC framework- Action-Perception Coupling

File: ros2_ws/src/cognibot_description/urdf/cognibot.urdf.xacro (robot description, xacro)
@@ -4,5 +4,6 @@
     <xacro:include filename="mobile_base.xacro"/>
     <!-- <xacro:include filename="mobile_base_ros2_control.xacro"/> -->
-    <xacro:include filename="camera.xacro"/>
+    <!-- <xacro:include filename="camera.xacro"/> -->
+    <xacro:include filename="lidar.xacro"/>
 <!--
     <xacro:include filename="camera.xacro"/>

File: ros2_ws/src/cognibot_description/urdf/common_properties.xacro (robot description, xacro)
@@ -20,4 +20,7 @@
     </material>
     <material name="camera">
+        <color rgba="1 1 0 1"/>
+    </material>
+    <material name="lidar">
         <color rgba="1 1 0 1"/>
     </material>

Commit message: Refactored code

File: ros2_ws/src/cognibot_description/urdf/cognibot.urdf.xacro (robot description, xacro)
@@ -3,15 +3,4 @@
     <xacro:include filename="common_properties.xacro"/>
     <xacro:include filename="mobile_base.xacro"/>
-    <!-- <xacro:include filename="mobile_base_ros2_control.xacro"/> -->
-    <!-- <xacro:include filename="camera.xacro"/> -->
     <xacro:include filename="lidar.xacro"/>
-<!--
-    <xacro:include filename="camera.xacro"/>
-    <xacro:include filename="arm.xacro"/>
-    <joint name = "arm_base_to_mobile_base_joint" type="fixed">
-        <parent link="base_link"/>
-        <child link="arm_base_link"/>
-        <origin xyz="${base_length/3.0} 0 ${base_height}" rpy="0 0 0"/>
-    </joint>
-     -->
 </robot>
